File: LM5143_Buck.kicad_sch (KiCad schematic)
At the start: 50 parts, among them Q1 BSC13DN30NSFD, Q2 BSC13DN30NSFD, Q3 BSC13DN30NSFD, Q4 BSC13DN30NSFD

Commit message: test
Other:
- note added: "test"
Changed lines of the file:
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@@
 	(generator_version "10.0")
 	(paper "A2")
+	(text "test"
+		(exclude_from_sim no)
+		(at 78.74 108.204 0)
+		(effects
+			(font
+				(size 1.27 1.27)
+			)
+		)
+	)
 	(junction
 		(at 359.41 105.41)
