File: Main_PDB.kicad_sch (KiCad schematic)
At the start: 124 parts, among them J1 Conn_01x02_MountingPin, J10 Conn_01x02_MountingPin, J12 Conn_01x02_MountingPin, J2 Conn_01x02_MountingPin, J3 Conn_01x02_MountingPin, J4 Conn_01x02_MountingPin, J5 Conn_01x02_MountingPin, J6 Conn_01x01_MountingPin, J7 Conn_01x01_MountingPin, J8 Conn_01x09_MountingPin, J9 Conn_01x03_MountingPin, Q1 PMOS, Q10 NMOS, Q14 NMOS, Q15 NMOS, Q2 NPN, Q7 NMOS, Q8 NMOS, Q9 NMOS, U1 LRM36015, U10 LM5148RGYR, U11 ACS758LCB-100U-PFF-T, U12 TPS48110AQDGXRQ1, U13 LM5148RGYR, U14 UCC27511DBVR, U2 ACS758LCB-100U-PFF-T, U4 ACS758LCB-100U-PFF-T, U5 ACS758LCB-100U-PFF-T, U6 ACS758LCB-100U-PFF-T, U8 ACS758LCB-100U-PFF-T, U9 ACS758LCB-100U-PFF-T

Commit message: caps
Parts:
- C14: value 83u -> 30u
- C2: value 285u -> 15u
Other:
- moved on the sheet: D7
Changed lines of the file:
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@@
 	)
 	(junction
-		(at 166.37 243.84)
+		(at 505.46 388.62)
 		(diameter 0)
 		(color 0 0 0 0)
 	)
 	(junction
-		(at 504.19 388.62)
+		(at 166.37 243.84)
 		(diameter 0)
 		(color 0 0 0 0)
@@
 	(wire
 		(pts
+			(xy 505.46 388.62) (xy 510.54 388.62)
+		)
+		(stroke
+			(width 0)
+			(type default)
+		)
+	)
+	(wire
+		(pts
 			(xy 64.77 138.43) (xy 64.77 114.3)
 		)
@@
 	(wire
 		(pts
-			(xy 499.11 388.62) (xy 504.19 388.62)
+			(xy 499.11 388.62) (xy 505.46 388.62)
 		)
 		(stroke
@@
 	(wire
 		(pts
-			(xy 504.19 388.62) (xy 510.54 388.62)
-		)
-		(stroke
-			(width 0)
-			(type default)
-		)
-	)
-	(wire
-		(pts
 			(xy 34.29 99.06) (xy 68.58 99.06)
 		)
@@
 	(symbol
 		(lib_id "Device:D_Zener")
-		(at 504.19 384.81 90)
+		(at 505.46 384.81 90)
 		(unit 1)
 		(body_style 1)
@@
 		(dnp no)
 		(property "Reference" "D7"
-			(at 508 382.27 90)
+			(at 509.27 382.27 90)
 			(show_name no)
 			(do_not_autoplace no)
@@
 		)
 		(property "Value" "TVS"
-			(at 508 384.81 90)
+			(at 509.27 384.81 90)
 			(show_name no)
 			(do_not_autoplace no)
@@
 		)
 		(property "Footprint" ""
-			(at 504.19 384.81 0)
+			(at 505.46 384.81 0)
 			(hide yes)
 			(show_name no)
@@
 		)
 		(property "Datasheet" ""
-			(at 504.19 384.81 0)
+			(at 505.46 384.81 0)
 			(hide yes)
 			(show_name no)
@@
 		)
 		(property "Description" "Zener diode"
-			(at 504.19 384.81 0)
+			(at 505.46 384.81 0)
 			(hide yes)
 			(show_name no)
@@
 	(symbol
 		(lib_id "power:GND")
-		(at 504.19 381 180)
+		(at 505.46 381 180)
 		(unit 1)
 		(body_style 1)
@@
 		(fields_autoplaced yes)
 		(property "Reference" "#PWR054"
-			(at 504.19 374.65 0)
+			(at 505.46 374.65 0)
 			(hide yes)
 			(show_name no)
@@
 		)
 		(property "Value" "GND"
-			(at 504.1901 377.19 90)
+			(at 505.4601 377.19 90)
 			(show_name no)
 			(do_not_autoplace no)
@@
 		)
 		(property "Footprint" ""
-			(at 504.19 381 0)
+			(at 505.46 381 0)
 			(hide yes)
 			(show_name no)
@@
 		)
 		(property "Datasheet" ""
-			(at 504.19 381 0)
+			(at 505.46 381 0)
 			(hide yes)
 			(show_name no)
@@
 		)
 		(property "Description" "Power symbol creates a global label with name \"GND\" , ground"
-			(at 504.19 381 0)
+			(at 505.46 381 0)
 			(hide yes)
 			(show_name no)
@@
 			)
 		)
-		(property "Value" "285u"
+		(property "Value" "15u"
 			(at 335.28 351.7899 0)
 			(show_name no)
@@
 			)
 		)
-		(property "Value" "83u"
+		(property "Value" "30u"
 			(at 502.92 393.6999 0)
 			(show_name no)
