File: Main_PDB.kicad_sch (KiCad schematic)
At the start: 128 parts, among them J1 Conn_01x02_MountingPin, J10 Conn_01x02_MountingPin, J12 Conn_01x02_MountingPin, J2 Conn_01x02_MountingPin, J3 Conn_01x02_MountingPin, J4 Conn_01x02_MountingPin, J5 Conn_01x02_MountingPin, J6 Conn_01x01_MountingPin, J7 Conn_01x01_MountingPin, J8 Conn_01x09_MountingPin, J9 Conn_01x03_MountingPin, Q1 PMOS, Q10 NMOS, Q14 NMOS, Q15 NMOS, Q2 NPN, Q7 NMOS, Q8 NMOS, Q9 NMOS, U1 LRM36015, U10 LM5148RGYR, U11 ACS758LCB-100U-PFF-T, U12 TPS48110AQDGXRQ1, U13 LM5148RGYR, U14 UCC27511DBVR, U2 ACS758LCB-100U-PFF-T, U4 ACS758LCB-100U-PFF-T, U5 ACS758LCB-100U-PFF-T, U6 ACS758LCB-100U-PFF-T, U8 ACS758LCB-100U-PFF-T, U9 ACS758LCB-100U-PFF-T

Commit message: Grounding and inductor and output caps on 12V buck
Parts:
- removed C48: 47u, symbol Device:C_Polarized
- removed R4: PullUpRes, symbol Device:R
- removed RPG1: 100KR, symbol Device:R_US
- added C48: 22u, symbol Device:C
- added J11: Conn_01x03_MountingPin, symbol Connector_Generic_MountingPin:Conn_01x03_MountingPin
- C46: value 4.7u -> 22u
- L5: value 1u -> 7.69u (30%)
- R17: value 54.4k -> 33k
- R18: value 40.2k -> 41.2k
Connections:
- net AGND: now also C34.2, C35.2, C36.2, C37.2, C50.1, C53.2, U12.10 (DIODE), U12.2 (OV), U12.6 (GND), U12.7 (IMON), U12.8 (IWRN), U12.9 (TMR), U14.4 (GND), U14.5 (IN-), U2.2 (GND), U4.2 (GND), U5.2 (GND), U6.2 (GND), U8.2 (GND); no longer C13.2, C14.2, C2.1, C26.2, C27.2, C28.2, C29.2, C3.2, C30.2, C31.2, C38.2, C39.2, C40.2, C41.2, C43.2, C44.2, C46.2, C49.2, C6.2, CHF1.2, CHF2.2, CIN1.2, J1.2 (Pin_2), J10.2 (Pin_2), Q15.3 (S), Q9.3 (S), R12.2, R21.2, U10.10 (PGND), U10.17 (PG/SYNCOUT), U10.25 (EP), U13.10 (PGND), U13.25 (EP)
- net GND: no longer C10.2, C11.2, C12.2, C19.2, C20.2, C21.2, C22.2, C23.2, C24.2, C7.2, C8.2, C9.2, D1.2 (A), D2.2 (A), D3.2 (A), D4.2 (A), D5.2 (A), J2.2 (Pin_2), J3.2 (Pin_2), J4.2 (Pin_2), J5.2 (Pin_2), Q2.3 (E), R1.2, U12.10 (DIODE), U12.2 (OV), U12.6 (GND), U12.7 (IMON), U12.8 (IWRN), U12.9 (TMR)
- net GND1: no longer C34.2, C35.2, C36.2, C37.2, C50.1, C53.2, U14.4 (GND), U14.5 (IN-), U2.2 (GND), U4.2 (GND), U5.2 (GND), U6.2 (GND), U8.2 (GND)
- net at C46.1, R20.1, R22.2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: now also C48.1
- removed net STM32: TH1.1, TH2.1, TH3.1
- new net: J11.1 (Pin_1), TH1.1
- new net: J11.3 (Pin_3), TH3.1
- new net: J11.2 (Pin_2), TH2.1
- new net PGND: C10.2, C11.2, C12.2, C13.2, C14.2, C19.2, C2.1, C20.2, C21.2, C22.2, C23.2, C24.2, C26.2, C27.2, C28.2, C29.2, C3.2, C30.2, C31.2, C38.2, C39.2, C40.2, C41.2, C43.2, C44.2, C46.2, C48.2, C49.2, C6.2, C7.2, C8.2, C9.2, CHF1.2, CHF2.2, CIN1.2, D1.2 (A), D2.2 (A), D3.2 (A), D4.2 (A), D5.2 (A), J1.2 (Pin_2), J10.2 (Pin_2), J2.2 (Pin_2), J3.2 (Pin_2), J4.2 (Pin_2), J5.2 (Pin_2), Q15.3 (S), Q2.3 (E), Q9.3 (S), R1.2, R12.2, R21.2, U10.10 (PGND), U10.25 (EP), U13.10 (PGND), U13.25 (EP)
- no-connect marks 12 -> 15
Other:
- note added: "SF-650.19 kHz"

Commit message: Added compute buck cap
Parts:
- removed J8: Conn_01x09_MountingPin, symbol Connector_Generic_MountingPin:Conn_01x09_MountingPin
- added C15: 220u, symbol Device:C_Polarized
- added J8: Conn_01x07_MountingPin, symbol Connector_Generic_MountingPin:Conn_01x07_MountingPin
Connections:
- net Act_rail_curr: now also J8.1 (Pin_1)
- net Com_cur: now also J8.7 (Pin_7)
- net GND: no longer D6.2 (A)
- net Main_curr: now also J8.6 (Pin_6)
- net PGND: now also D6.2 (A), C15.2
- net at U6.3 (VIOUT): now also J8.2 (Pin_2)
- net at U4.3 (VIOUT): now also J8.4 (Pin_4)
- net at U5.3 (VIOUT): now also J8.3 (Pin_3)
- net at U2.3 (VIOUT): now also J8.5 (Pin_5)
- net at D8.1 (K), J1.1 (Pin_1), U11.5 (IP-)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: now also C15.1
