File: Main_PDB.kicad_pcb (KiCad board)
At the start: 4 copper layers, 175.5 x 85.5 mm, 134 parts, among them Q4 NMOS, Q5 NMOS, Q6 NMOS, Q7 NMOS, Q8 NMOS, U10 ACS758LCB-100U-PFF-T, U11 ACS758LCB-100U-PFF-T, U12 ACS758LCB-100U-PFF-T, U2 LM5148RGYR, U3 LMR36015ARNXR, U4 ACS758LCB-100U-PFF-T, U5 ACS758LCB-100U-PFF-T, U6 UCC27511DBVR, U8 ACS758LCB-100U-PFF-T, U9 ACS758LCB-100U-PFF-T

Commit message: sorted components for 12V buck
Parts:
- moved U2 281.3 mm to (343.5, 179.5)
- moved COUT1B1 275.0 mm to (321.0, 179.0)
- moved COUT2B1 268.6 mm to (322.0, 161.0)
- moved COUT3B1 268.6 mm to (322.0, 169.5)
- moved CIN1B1 251.4 mm to (309.0, 203.5)
- moved CIN2B1 251.4 mm to (287.2, 158.7)
- moved CIN3B1 251.4 mm to (287.2, 167.2)
- moved CIN4B1 251.4 mm to (287.2, 175.7)
- moved RFB1 251.4 mm to (305.5, 159.0)
- moved RFB1A1 250.8 mm to (305.5, 163.0)
- moved COUT4B1 246.8 mm to (311.1, 160.5)
- moved RFB2B1 5.94 mm to (100.5, 30.0)
- moved RPD1 5.94 mm to (100.5, 34.8)
Changed lines of the file:
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@@
 	(footprint "Capacitor_SMD:C_1210_3225Metric"
 		(layer "F.Cu")
-		(at 57.795 64.475)
+		(at 287.235 167.2)
 		(descr "Capacitor SMD 1210 (3225 Metric), square (rectangular) end terminal, IPC-7351 nominal, (Body size source: IPC-SM-782 page 76, https://www.pcb-3d.com/wordpress/wp-content/uploads/ipc-sm-782a_amendment_1_and_2.pdf)")
 		(tags "capacitor")
@@
 	(footprint "Resistor_SMD:R_0603_1608Metric"
 		(layer "F.Cu")
-		(at 94.565 27.275)
+		(at 305.5 163)
 		(descr "Resistor SMD 0603 (1608 Metric), square (rectangular) end terminal, IPC-7351 nominal, (Body size source: IPC-SM-782 page 72, https://www.pcb-3d.com/wordpress/wp-content/uploads/ipc-sm-782a_amendment_1_and_2.pdf)")
 		(tags "resistor")
@@
 	(footprint "Capacitor_SMD:C_1210_3225Metric"
 		(layer "F.Cu")
-		(at 74.745 64.475)
+		(at 322 169.5)
 		(descr "Capacitor SMD 1210 (3225 Metric), square (rectangular) end terminal, IPC-7351 nominal, (Body size source: IPC-SM-782 page 76, https://www.pcb-3d.com/wordpress/wp-content/uploads/ipc-sm-782a_amendment_1_and_2.pdf)")
 		(tags "capacitor")
@@
 	(footprint "Capacitor_SMD:C_0805_2012Metric"
 		(layer "F.Cu")
-		(at 84.245 63.145)
+		(at 311.05 160.5)
 		(descr "Capacitor SMD 0805 (2012 Metric), square (rectangular) end terminal, IPC-7351 nominal, (Body size source: IPC-SM-782 page 76, https://www.pcb-3d.com/wordpress/wp-content/uploads/ipc-sm-782a_amendment_1_and_2.pdf, https://docs.google.com/spreadsheets/d/1BsfQQcO9C6DZCsRaXUlFlo91Tg2WpOkGARC1WS5S8t0/edit?usp=sharing)")
 		(tags "capacitor")
@@
 	(footprint "Capacitor_SMD:C_1210_3225Metric"
 		(layer "F.Cu")
-		(at 74.745 55.975)
+		(at 322 161)
 		(descr "Capacitor SMD 1210 (3225 Metric), square (rectangular) end terminal, IPC-7351 nominal, (Body size source: IPC-SM-782 page 76, https://www.pcb-3d.com/wordpress/wp-content/uploads/ipc-sm-782a_amendment_1_and_2.pdf)")
 		(tags "capacitor")
@@
 	(footprint "Footprints:QFN50P550X350X100-25N"
 		(layer "F.Cu")
-		(at 81.015 78.36)
+		(at 343.5 179.5)
 		(property "Reference" "U2"
 			(at -0.485 -5 0)
@@
 	(footprint "Capacitor_SMD:CP_Elec_10x10"
 		(layer "F.Cu")
-		(at 79.56 100.775)
+		(at 309 203.5)
 		(descr "SMD capacitor, aluminum electrolytic, Nichicon, 10.0x10.0mm")
 		(tags "capacitor electrolytic")
@@
 	(footprint "Capacitor_SMD:C_1210_3225Metric"
 		(layer "F.Cu")
-		(at 69.095 68.725)
+		(at 321.025 179)
 		(descr "Capacitor SMD 1210 (3225 Metric), square (rectangular) end terminal, IPC-7351 nominal, (Body size source: IPC-SM-782 page 76, https://www.pcb-3d.com/wordpress/wp-content/uploads/ipc-sm-782a_amendment_1_and_2.pdf)")
 		(tags "capacitor")
@@
 	(footprint "Resistor_SMD:R_0603_1608Metric"
 		(layer "F.Cu")
-		(at 94.565 22.255)
+		(at 305.5 159)
 		(descr "Resistor SMD 0603 (1608 Metric), square (rectangular) end terminal, IPC-7351 nominal, (Body size source: IPC-SM-782 page 72, https://www.pcb-3d.com/wordpress/wp-content/uploads/ipc-sm-782a_amendment_1_and_2.pdf)")
 		(tags "resistor")
@@
 	(footprint "Capacitor_SMD:C_1210_3225Metric"
 		(layer "F.Cu")
-		(at 57.795 72.975)
+		(at 287.235 175.7)
 		(descr "Capacitor SMD 1210 (3225 Metric), square (rectangular) end terminal, IPC-7351 nominal, (Body size source: IPC-SM-782 page 76, https://www.pcb-3d.com/wordpress/wp-content/uploads/ipc-sm-782a_amendment_1_and_2.pdf)")
 		(tags "capacitor")
@@
 	(footprint "Capacitor_SMD:C_1210_3225Metric"
 		(layer "F.Cu")
-		(at 57.795 55.975)
+		(at 287.235 158.7)
 		(descr "Capacitor SMD 1210 (3225 Metric), square (rectangular) end terminal, IPC-7351 nominal, (Body size source: IPC-SM-782 page 76, https://www.pcb-3d.com/wordpress/wp-content/uploads/ipc-sm-782a_amendment_1_and_2.pdf)")
 		(tags "capacitor")
@@
 	(footprint "Resistor_SMD:R_0603_1608Metric"
 		(layer "F.Cu")
-		(at 94.565 29.785)
+		(at 100.5 30)
 		(descr "Resistor SMD 0603 (1608 Metric), square (rectangular) end terminal, IPC-7351 nominal, (Body size source: IPC-SM-782 page 72, https://www.pcb-3d.com/wordpress/wp-content/uploads/ipc-sm-782a_amendment_1_and_2.pdf)")
 		(tags "resistor")
@@
 	(footprint "Resistor_SMD:R_0603_1608Metric"
 		(layer "F.Cu")
-		(at 94.565 34.805)
+		(at 100.5 34.805)
 		(descr "Resistor SMD 0603 (1608 Metric), square (rectangular) end terminal, IPC-7351 nominal, (Body size source: IPC-SM-782 page 72, https://www.pcb-3d.com/wordpress/wp-content/uploads/ipc-sm-782a_amendment_1_and_2.pdf)")
 		(tags "resistor")
