File: Main_PDB.kicad_pcb (KiCad board)
At the start: 4 copper layers, 175.5 x 234.8 mm, 155 parts, among them J10 Conn_01x02_MountingPin, J5 24V Out -> Jetson, J6 24V Out -> USB-C-PD controller, J7 Conn_01x02_MountingPin, J8 Conn_01x02_MountingPin, J9 Conn_01x02_MountingPin, Q4 NMOS, Q5 NMOS, Q6 NMOS, Q7 NMOS, Q8 NMOS, U1 TLV3011AIDBVT, U10 ACS758LCB-100U-PFF-T, U11 ACS758LCB-100U-PFF-T, U12 ACS758LCB-100U-PFF-T, U2 LM5148RGYR, U3 LMR36015ARNXR, U4 ACS758LCB-100U-PFF-T, U5 ACS758LCB-100U-PFF-T, U6 UCC27511DBVR, U8 ACS758LCB-100U-PFF-T, U9 ACS758LCB-100U-PFF-T

Commit message: fixed merge
Parts:
- removed RFBS1: 49.9k, Resistor_SMD:R_0603_1608Metric
- added J5: 24V Out -> Jetson, Connector_Phoenix_MC:PhoenixContact_MC_1,5_2-G-3.81_1x02_P3.81mm_Horizontal, F.Cu at (387.5, 143.1)
- added J6: 24V Out -> USB-C-PD controller, Connector_Phoenix_MC:PhoenixContact_MC_1,5_2-G-3.81_1x02_P3.81mm_Horizontal, F.Cu at (387.5, 153.8)
- moved CIN1B1 234.5 mm to (432.0, 124.6), turned to 90 degrees
- moved CIN4B1 230.1 mm to (424.7, 125.8), turned to -90 degrees
- moved CIN3B1 229.0 mm to (421.4, 125.8), turned to -90 degrees
- moved CIN2B1 228.0 mm to (418.1, 125.8), turned to -90 degrees
- moved CIN5B1 226.4 mm to (415.4, 126.3), turned to -90 degrees
- moved F2 225.2 mm to (440.2, 134.2), turned to 180 degrees
- moved RFB1A2 223.6 mm to (407.9, 127.1), turned to 0 degrees
- moved RFB2B2 221.8 mm to (401.1, 126.2), turned to 0 degrees
- moved RCON1 221.6 mm to (401.1, 127.7), turned to 0 degrees
- moved RSF1 219.4 mm to (401.1, 129.2), turned to 0 degrees
- moved RCOMP1 218.8 mm to (403.4, 129.9), turned to -90 degrees
- moved RSEN1 218.3 mm to (427.4, 135.2), turned to -90 degrees
- moved CCOMP1 217.3 mm to (401.1, 130.7), turned to 180 degrees
- moved L2 216.4 mm to (420.7, 134.8), turned to 90 degrees
- moved Q4 215.9 mm to (413.3, 133.5), turned to -90 degrees
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Connections:
- net /12V_FUSE renamed /24V_FUSE
- net /12V_IND renamed /24V_IND
- net /12V_NMOS renamed /24V_SW
- net /12V_SEN renamed /24V_SEN
Routing:
- net Net-(U2-VDDA): track 8.62 -> 1.54 mm, vias 2 -> 1
- net Net-(U2-FB): track 9.41 -> 13.5 mm, vias 2 -> 3
- net AGND: track 61.6 -> 59.1 mm
- removed copper zone on F.Cu, net (none)

Commit message: Placement for current sen signal pass
Parts:
- moved CCS6 483.3 mm to (504.0, 258.8)
- moved CCSF6 474.6 mm to (504.8, 256.4), turned to 90 degrees
- moved RCSF6 468.0 mm to (504.0, 254.0)
- moved CCS7 466.9 mm to (504.2, 225.2)
- moved CCSF7 459.4 mm to (505.0, 222.8), turned to 90 degrees
- moved RCSF7 452.4 mm to (504.2, 220.4)
- moved CCS8 449.3 mm to (504.2, 182.4)
- moved CCSF8 443.6 mm to (505.0, 180.0), turned to 90 degrees
- moved RCSF8 436.0 mm to (504.2, 177.6)
- moved CCS5 432.8 mm to (450.4, 266.2)
- moved CCSF5 432.6 mm to (451.2, 263.6), turned to 90 degrees
- moved RCSF5 426.4 mm to (450.4, 261.0)

Commit message: output caps on 24V rail footprint update
Parts:
- added COUT4B1: 100nF, Capacitor_SMD:C_0603_1608Metric, F.Cu at (430.0, 150.0)
- moved COUT4B1 104.8 mm to (523.4, 102.3)
Connections:
- U6 pad 5: AGND -> Net-(U1-OUT)
- U6 pad 6: Net-(U1-OUT) -> AGND

Commit message: Minor layout change
Parts:
- removed the COUT4B1 at (523.4, 102.3)
Changed lines of the file:
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@@
-		)
-	)
-	(footprint "Capacitor_SMD:C_0805_2012Metric"
-		(layer "F.Cu")
-		(at 523.383156 102.270939)
-		(descr "Capacitor SMD 0805 (2012 Metric), square (rectangular) end terminal, IPC-7351 nominal, (Body size source: IPC-SM-782 page 76, https://www.pcb-3d.com/wordpress/wp-content/uploads/ipc-sm-782a_amendment_1_and_2.pdf, https://docs.google.com/spreadsheets/d/1BsfQQcO9C6DZCsRaXUlFlo91Tg2WpOkGARC1WS5S8t0/edit?usp=sharing)")
-		(tags "capacitor")
-		(property "Reference" "COUT4B1"
-			(at 0 -1.68 0)
-			(layer "F.SilkS")
-			(effects
-				(font
-					(size 1 1)
-					(thickness 0.15)
-				)
-			)
-		)
-		(property "Value" "100nF"
-			(at 0 1.68 0)
-			(layer "F.Fab")
-			(effects
-				(font
-					(size 1 1)
-					(thickness 0.15)
-				)
-			)
-		)
-		(property "Datasheet" ""
-			(at 0 0 0)
-			(layer "F.Fab")
-			(hide yes)
-			(effects
-				(font
-					(size 1.27 1.27)
-				)
-			)
-		)
-		(property "Description" "Unpolarized capacitor XR7"
-			(at 0 0 0)
-			(layer "F.Fab")
-			(hide yes)
-			(effects
-				(font
-					(size 1.27 1.27)
-				)
-			)
-		)
-		(property "KiLib_Generator" "SMD_2terminal_chip_molded"
-			(at 0 0 0)
-			(layer "F.SilkS")
-			(hide yes)
-			(effects
-				(font
-					(size 1 1)
-					(thickness 0.15)
-				)
-			)
-		)
-		(property "Voltage" "25V"
-			(at 0 0 0)
-			(unlocked yes)
-			(layer "F.Fab")
-			(hide yes)
-			(effects
-				(font
-					(size 1 1)
-					(thickness 0.15)
-				)
-			)
-		)
-		(property ki_fp_filters "C_*")
-		(sheetname "/")
-		(sheetfile "Main_PDB.kicad_sch")
-		(attr smd)
-		(duplicate_pad_numbers_are_jumpers no)
-		(fp_line
-			(start -0.261252 -0.735)
-			(end 0.261252 -0.735)
-			(stroke
-				(width 0.12)
-				(type solid)
-			)
-			(layer "F.SilkS")
-		)
-		(fp_line
-			(start -0.261252 0.735)
-			(end 0.261252 0.735)
-			(stroke
-				(width 0.12)
-				(type solid)
-			)
-			(layer "F.SilkS")
-		)
-		(fp_rect
-			(start -1.7 -0.98)
-			(end 1.7 0.98)
-			(stroke
-				(width 0.05)
-				(type solid)
-			)
-			(fill no)
-			(layer "F.CrtYd")
-		)
-		(fp_rect
-			(start -1 -0.625)
-			(end 1 0.625)
-			(stroke
-				(width 0.1)
-				(type solid)
-			)
-			(fill no)
-			(layer "F.Fab")
-		)
-		(fp_text user "${REFERENCE}"
-			(at 0 0 0)
-			(layer "F.Fab")
-			(effects
-				(font
-					(size 0.5 0.5)
-					(thickness 0.08)
-				)
-			)
-		)
-		(pad "1" smd roundrect
-			(at -0.95 0)
-			(size 1 1.45)
-			(layers "F.Cu" "F.Mask" "F.Paste")
-			(roundrect_rratio 0.25)
-			(net "/24V_SEN")
-			(pintype "passive")
-		)
-		(pad "2" smd roundrect
-			(at 0.95 0)
-			(size 1 1.45)
-			(layers "F.Cu" "F.Mask" "F.Paste")
-			(roundrect_rratio 0.25)
-			(net "PGND")
-			(pintype "passive")
-		)
-		(embedded_fonts no)
-		(model "${KICAD10_3DMODEL_DIR}/Capacitor_SMD.3dshapes/C_0805_2012Metric.step"
-			(offset
-				(xyz 0 0 0)
-			)
-			(scale
-				(xyz 1 1 1)
-			)
-			(rotate
-				(xyz 0 0 0)
-			)
 		)
 	)

Commit message: 6V Buck layout finished
Parts:
- added CCS9: 100n, Capacitor_SMD:C_0603_1608Metric, F.Cu at (1.50, 0.76)
- added U7: LM5148RGYR, Footprints:QFN50P550X350X100-25N, F.Cu at (406.5, 188.4)
- CCOMP2: value 6.8nF -> 4.7nF
- RCOMP2: value 4.75k -> 6.49k
- RPRE1: value 80R -> R
- moved CIN4B2 383.4 mm to (424.5, 180.9), turned to -90 degrees
- moved CIN2B2 382.9 mm to (421.2, 180.9), turned to -90 degrees
- moved COUT1B2 379.4 mm to (424.8, 205.0), turned to -90 degrees
- moved COUT3B2 378.6 mm to (428.0, 205.0), turned to -90 degrees
- moved D8 377.6 mm to (405.4, 205.7), turned to -90 degrees
- moved CIN3B2 377.1 mm to (417.9, 180.9), turned to -90 degrees
- moved COUT2B2 375.7 mm to (421.5, 205.0), turned to -90 degrees
- moved CBOOT3 369.4 mm to (409.7, 191.0), turned to 90 degrees
- moved RSEN2 365.3 mm to (427.5, 190.4), turned to -90 degrees
- moved CBULK2 361.0 mm to (414.3, 205.7), turned to -90 degrees
- moved CIN1B2 358.6 mm to (431.8, 179.8), turned to 90 degrees
- moved CCOMP2 357.2 mm to (401.0, 186.0), turned to 180 degrees
- moved CIN5B2 355.7 mm to (415.3, 181.5), turned to -90 degrees
- moved CHF2 354.3 mm to (402.5, 187.5), turned to 180 degrees
- moved CVDDA2 351.7 mm to (402.5, 189.3)
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Connections:
- net /24V_SW renamed /24V_NMOS
Routing:
- net +6V: track 0.00 -> 24.3 mm, vias 0 -> 2
- net AGND: track 59.1 -> 73.8 mm, vias 3 -> 5
- net Net-(U7-FB): track 0.00 -> 13.5 mm, vias 0 -> 2
- net /6V_FUSE: track 0.00 -> 12.2 mm, vias 0 -> 2
- net +6V_IND: track 0.00 -> 9.17 mm, vias 0 -> 2
- net Net-(Q7-G): track 0.00 -> 8.92 mm, vias 0 -> 2
- net Net-(Q8-G): track 0.00 -> 8.09 mm
- net Net-(U7-CNFG): track 0.00 -> 5.11 mm, vias 0 -> 1
- net Net-(U7-EXTCOMP): track 0.00 -> 4.65 mm, vias 0 -> 2
- net Net-(U7-RT): track 0.00 -> 4.18 mm, vias 0 -> 1
- net Net-(U7-VCC): track 0.00 -> 2.87 mm
- net /6V_NMOS: track 0.00 -> 1.84 mm, vias 0 -> 16
- net Net-(CCOMP2-Pad1): track 0.00 -> 1.55 mm
- net Net-(U7-VDDA): track 0.00 -> 1.54 mm, vias 0 -> 1
- net PGND: vias 62 -> 84
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- added copper zone on F.Cu, net +6V
- added copper zone on F.Cu, net +6V_IND
- added copper zone on F.Cu, net /6V_FUSE
- added copper zone on F.Cu, net /6V_NMOS

Commit message: small routing
Parts:
- removed the J5 at (114.2, 25.9)
- removed the J6 at (125.4, 25.9)
- removed RESTOP1, RESTOP2: 100, Resistor_SMD:R_0603_1608Metric
- removed RESTOP3: 4.3k 1W, Resistor_SMD:R_0603_1608Metric
- removed RESTOP4: 10k, Resistor_SMD:R_0603_1608Metric
- removed RPD1, RPU1: 10K, Resistor_SMD:R_0603_1608Metric
- added CCS10: 100uF 50V, Capacitor_SMD:CP_Elec_6.3x5.4, F.Cu at (346.5, 148.0)
- added CCS11: 100nF 50V, Capacitor_SMD:C_0603_1608Metric, F.Cu at (363.0, 147.7)
- added CCS12: 100nF 50V, Capacitor_SMD:C_0603_1608Metric, F.Cu at (354.4, 147.5)
- added D9: 12V Zener 1W, Diode_SMD:D_SMA, F.Cu at (355.0, 156.5)
- added F1: Fuse, Footprints:FUSE_2822HC100-RTR, F.Cu at (344.0, 55.0)
- added J2: Rockchip ESTOP feedback, Connector_PinHeader_1.00mm:PinHeader_1x01_P1.00mm_Vertical, F.Cu at (337.8, 148.1)
- added J20: ESTOP Contactor Coil Control, TerminalBlock:TerminalBlock_MaiXu_MX126-5.0-02P_1x02_P5.00mm, F.Cu at (341.0, 118.8)
- added J21: ESTOP Button (Normally Closed), TerminalBlock:TerminalBlock_MaiXu_MX126-5.0-02P_1x02_P5.00mm, F.Cu at (341.0, 134.0)
- added J23: Rockchip FET Control, Connector_PinHeader_1.00mm:PinHeader_1x02_P1.00mm_Vertical, F.Cu at (337.8, 143.9)
- added Q2: NMOS IRFR220N, Package_TO_SOT_SMD:TO-252-3_TabPin2, F.Cu at (353.8, 130.9)
- added Q3: NMOS IRFR220N, Package_TO_SOT_SMD:TO-252-3_TabPin2, F.Cu at (362.2, 130.8)
- added RESTP1: 10, Resistor_SMD:R_0603_1608Metric, F.Cu at (353.7, 139.5)
- added RESTP2: 10, Resistor_SMD:R_0603_1608Metric, F.Cu at (362.4, 139.5)
- added RESTP3: 10K, Resistor_SMD:R_0603_1608Metric, F.Cu at (362.5, 151.5)
- added RESTP4: 10K, Resistor_SMD:R_0603_1608Metric, F.Cu at (354.5, 151.5)
- added RESTP5: TBD R, Resistor_SMD:R_0603_1608Metric, F.Cu at (341.7, 156.5)
- added RESTP6: TBD R, Resistor_SMD:R_0603_1608Metric, F.Cu at (347.5, 156.5)
- added RESTP7: 4.7K 1W, Resistor_SMD:R_2512_6332Metric, F.Cu at (364.0, 157.0)
- added U13: MCP1401T-E/OT, Footprints:SOT-23-5_MC_MCH, F.Cu at (354.5, 144.2)
- added U14: MCP1401T-E/OT, Footprints:SOT-23-5_MC_MCH, F.Cu at (363.0, 144.2)
- D10: value TVS -> TVS 93.6V max clamp; footprint Diode_SMD:D_SMC -> Diode_SMD:D_SMB
- moved D10 246.0 mm to (348.6, 121.2), turned to -90 degrees
- moved CCS9 125.7 mm to (114.5, 55.8)
- moved D1 78.8 mm to (122.0, 55.9)
- moved D2 78.8 mm to (122.0, 63.6)
- moved RFB2 45.6 mm to (114.5, 65.8)
- moved U6 41.9 mm to (130.6, 58.7)
- moved COUT4B2 41.9 mm to (126.6, 69.0)
- moved Q6 41.7 mm to (120.4, 70.9)
- moved RPRE1 39.0 mm to (114.5, 70.8)
- moved RDIV1 34.8 mm to (114.5, 58.3)
- moved RFBC1 34.8 mm to (114.5, 68.3)
- moved RDIV2 34.8 mm to (114.5, 60.8)
- moved CCS3 29.0 mm to (114.5, 53.3)
- moved U1 24.0 mm to (130.6, 54.2)
- moved RFB1 24.0 mm to (114.5, 63.3)
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Routing:
- net /48V_FUSE: track 0.00 -> 53.3 mm, vias 0 -> 2
- net Net-(D9-K): track 0.00 -> 39.2 mm
- net Net-(J23-Pin_1): track 0.00 -> 34.6 mm, vias 0 -> 2
- net Net-(J23-Pin_2): track 0.00 -> 27.5 mm, vias 0 -> 2
- net Net-(J21-Pin_2): track 0.00 -> 21.5 mm
- net Net-(D10-A): track 0.00 -> 18.0 mm
- net Net-(J2-Pin_1): track 0.00 -> 14.5 mm
- net Net-(Q2-S): track 0.00 -> 13.6 mm
- net Net-(Q3-G): track 0.00 -> 3.91 mm
- net Net-(Q2-G): track 0.00 -> 3.70 mm
- net Net-(U14-*OUT): track 0.00 -> 2.73 mm
Other:
- board text added: "BTN"
- board text added: "COIL"

Commit message: Layout changes
Parts:
- moved COUT4B2 299.4 mm to (374.9, 236.2), turned to -90 degrees
- moved JESTOP1 33.7 mm to (471.0, 108.5)
- moved JESTOP2 33.7 mm to (471.0, 124.8)
- moved U6 30.7 mm to (131.2, 89.4)
- moved U1 30.7 mm to (131.2, 84.9)
- moved CBOOT1 28.0 mm to (384.5, 167.5)
- moved CIN2B2 28.0 mm to (395.9, 212.7)
- moved COUT3B1 28.0 mm to (405.1, 179.1)
- moved F3 28.0 mm to (414.9, 221.3)
- moved Q4 28.0 mm to (388.0, 165.4)
- moved RCSF1 28.0 mm to (394.2, 206.0)
- moved RFB2B2 28.0 mm to (375.8, 158.0)
- moved U2 28.0 mm to (381.3, 165.0)
- moved U5 28.0 mm to (392.3, 192.8)
- moved CBOOT3 28.0 mm to (384.4, 222.8)
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Routing:
- added copper zone on F.Cu, net /48V_ESTOP

Commit message: Power pour topology update (layers tbd)
Parts:
- moved JESTOP1 22.2 mm to (493.2, 108.8)
- moved JESTOP2 22.2 mm to (493.2, 125.1)
- moved CBLKA1 15.8 mm to (417.0, 247.5), turned to 180 degrees
- moved CINC1 7.80 mm to (417.8, 256.3), turned to 0 degrees
- moved D5 6.82 mm to (414.2, 269.2), turned to 180 degrees
- moved J8 6.47 mm to (395.3, 270.1)
- moved CINC2 5.30 mm to (417.7, 260.2)
- moved CINC9 5.30 mm to (418.3, 263.4)
Routing:
- added copper zone on B.Cu, net /48V_ACT
- added copper zone on F.Cu, net /48V_ACT
